File: Hardware/Bit32F0.kicad_pcb (KiCad board)
At the start: 4 copper layers, 27 x 18.7 mm, 19 parts, among them J1 USB_C_Receptacle_USB2.0_16P, J2 Conn_01x09, J3 Conn_01x09, J4 Conn_01x04, U1 STM32F042F6Px, U2 LP5912-3.3DRV

Commit message: Added pictures
Other:
- board text added: "Bit32F042F6Px"
- board text added: "and the universe said I love you because you are love. And the game was over and the player woke up from the dream. And the player began a new dream. And the player dreamed again, dreamed better. And the player was the universe. And the player was love."
- board text added: "by Fynr1x"
- board text added: "{dblquote}We will show them Our signs in the horizons and within themselves{dblquote} (41:53)"
- board text removed: "Bit32 > faizeenhoque.dev"
- board text removed: "The universe loves you"
